File: ee/ovrdrive/ovrdrive.kicad_pcb (KiCad board)
At the start: 4 copper layers, 36.4 x 15 mm, 54 parts, among them J2 USB3_A, J4 Micro_SD_Card_Det_Hirose_DM3AT, SW1 SW_Push, U1 CH569W, U2 TLV62569DBV, U3 TLV62569DBV, Y2 30Mhz

Commit message: Hardware r1.0-rc1
Parts:
- added U5: TPD2EUSB30, Package_TO_SOT_SMD:Texas_DRT-3, F.Cu at (139.3, 107.2)
- added U6: TPD2EUSB30, Package_TO_SOT_SMD:Texas_DRT-3, F.Cu at (139.3, 101.2)
- added U7: TPD2EUSB30, Package_TO_SOT_SMD:Texas_DRT-3, B.Cu at (137.2, 105.7)
- C1, C6: value 22uF -> 4.7uF
Routing:
- net +1V2: track 29.0 -> 28.5 mm, vias 7 -> 6
- net GND: vias 87 -> 85
Other:
- board text added: "R1.0"
