File: ee/ovrdrive/ovrdrive.kicad_pcb (KiCad board)
At the start: 4 copper layers, 36.4 x 15 mm, 57 parts, among them J2 USB3_A, J4 Micro_SD_Card_Det_Hirose_DM3AT, SW1 SW_Push, U1 CH569W, U2 TLV62569DBV, U3 TLV62569DBV, U5 TPD2EUSB30, U6 TPD2EUSB30, U7 TPD2EUSB30, Y2 30Mhz

Commit message: Hardware r1.0 release.
Routing:
- net +3V3: track 27.0 -> 28.0 mm
- added copper zone on In2.Cu, net GND
Changed lines of the file:
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@@
 	)
 	(segment
+		(start 133.064869 106.423456)
+		(end 132.626544 106.423456)
+		(width 0.1)
+		(layer "In2.Cu")
+		(net "+3V3")
+	)
+	(segment
+		(start 132.65 101.2)
+		(end 132.6 101.15)
+		(width 0.1)
+		(layer "In2.Cu")
+		(net "+3V3")
+	)
+	(segment
+		(start 133.1 101.2)
+		(end 132.65 101.2)
+		(width 0.1)
+		(layer "In2.Cu")
+		(net "+3V3")
+	)
+	(segment
+		(start 132.626544 106.423456)
+		(end 132.6 106.45)
+		(width 0.1)
+		(layer "In2.Cu")
+		(net "+3V3")
+	)
+	(segment
 		(start 119.18 104)
 		(end 119.28 103.9)
@@
 	(zone
 		(net "GND")
-		(layers "F.Cu" "B.Cu" "In1.Cu")
+		(layers "F.Cu" "B.Cu" "In1.Cu" "In2.Cu")
 		(hatch edge 0.508)
 		(connect_pads thru_hole_only
@@
 		(polygon
 			(pts
-				(xy 120.9 98.3) (xy 120.9 104.2) (xy 130.1 104.2) (xy 130.1 109.7) (xy 133.2 109.7) (xy 133.2 98.205385)
+				(xy 120.9 98.3) (xy 120.9 104.2) (xy 130.1 104.2) (xy 130.1 109.7) (xy 132.8 109.7) (xy 132.8 98.208462)
 			)
 		)
