File: ee/ovrdrive/ovrdrive.kicad_sch (KiCad schematic)
At the start: 54 parts, among them J2 USB3_A, J4 Micro_SD_Card_Det_Hirose_DM3AT, SW1 SW_Push, U1 CH569W, U2 TLV62569DBV, U3 TLV62569DBV, Y2 30Mhz

Commit message: Hardware r1.0-rc1
Parts:
- added U5, U6, U7: TPD2EUSB30, Package_TO_SOT_SMD:Texas_DRT-3, symbol Power_Protection:TPD2EUSB30
- C1, C6: value 22uF -> 4.7uF; MPN CL05A226MQ5N6J8 -> CL05A475MP5NRNC
- C13, C2, C5: now not fitted
- J2: MPN 692112030100 -> XUSM-0930-231
Connections:
- net GND: now also U5.3 (GND), U6.3 (GND), U7.3 (GND)
- net USB_D+: now also U7.1 (D+)
- net USB_D-: now also U7.2 (D-)
- net USB_SSRX+: now also U6.2 (D-)
- net USB_SSRX-: now also U6.1 (D+)
- net USB_SSTX_R+: now also U5.2 (D-)
- net USB_SSTX_R-: now also U5.1 (D+)
Other:
- moved on the sheet: C3, C4, TP1, TP2, TP3
