File: ee/ovrdrive/ovrdrive.kicad_sch (KiCad schematic)
At the start: 57 parts, among them J2 USB3_A, J4 Micro_SD_Card_Det_Hirose_DM3AT, SW1 SW_Push, U1 CH569W, U2 TLV62569DBV, U3 TLV62569DBV, U5 TPD2EUSB30, U6 TPD2EUSB30, U7 TPD2EUSB30, Y2 30Mhz

Commit message: Hardware r1.0 release.
Other:
- title: Overdrive V2 -> Phantomdrive
Changed lines of the file:
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@@
 	(paper "A4")
 	(title_block
-		(title "Overdrive V2")
-		(date "2026-03-19")
-		(rev "R0.1")
+		(title "Phantomdrive")
+		(date "2026-03-29")
+		(rev "R1.0")
 		(company "Rootkit Labs")
 		(comment 1 "Ryan Walker")
